File: Serene Mini Hardware/Serene Mini.kicad_pcb (KiCad board)
At the start: 6 copper layers, 25 x 42.5 mm, 79 parts, among them J1 Conn_Coaxial, J2 Conn_01x06_Socket, J3 Conn_01x02, J4 AudioJack3_Switch, J5 USB_C_Receptacle_USB2.0_14P, J6 Conn_Coaxial, T1 Transformer_1P_1S, U1 AP7361C-33E, U2 AP2112K-1.8, U3 STM32H753ZITx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

Commit message: Changed Footprint
Added cooling and repositioned the testpoint pads to be closer ti each other
Parts:
- moved TP3 16.0 mm to (23.5, 53.2)
- moved TP1 15.8 mm to (23.5, 51.1)
- moved TP4 7.69 mm to (26.5, 51.8)
Routing:
- net /SWDIO: track 12.0 -> 8.08 mm
- net Net-(U6-TS_BIAS): track 5.26 -> 3.28 mm, vias 2 -> 0
- net /BTN_SENSE: track 43.3 -> 42.0 mm, vias 3 -> 5
- net /CHG_STAT: track 9.78 -> 11.0 mm, vias 3 -> 4
- net Net-(U6-TS): track 4.88 -> 3.75 mm, vias 0 -> 2
- net Net-(J3-Pin_1): track 18.1 -> 19.1 mm
- net GND: track 112.0 -> 111.4 mm, vias 92 -> 91
- net +3.3V: track 65.4 -> 64.9 mm
