File: Serene Mini Hardware/Serene Mini.kicad_pcb (KiCad board)
At the start: 6 copper layers, 25 x 42.5 mm, 80 parts, among them J1 Conn_Coaxial, J2 Conn_01x06_Socket, J4 AudioJack3_Switch, J5 USB_C_Receptacle_USB2.0_14P, J6 Conn_Coaxial, T1 Transformer_1P_1S, U1 AP7361C-33E, U2 AP2112K-1.8, U3 STM32H753ZITx, U4 ADXL382-1BCCZ-RL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

Commit message: Minor Changes
Parts:
- removed R12: 100kΩ, Resistor_SMD:R_0402_1005Metric
- added L3: 600Ω, Inductor_SMD:L_0402_1005Metric, F.Cu at (45.1, 66.2)
- added L4: 600Ω, Inductor_SMD:L_0402_1005Metric, F.Cu at (39.5, 54.0)
- C17: value 0.1uF -> 4.7µF
- R6: value 160Ω -> 170Ω
- U9: value ~ -> SR1120
- moved C20 1.35 mm to (45.1, 62.9), turned to 90 degrees
- moved C17 1.08 mm to (44.1, 66.2)
- moved C8 0.96 mm to (44.0, 64.3), turned to 90 degrees
- turned R4 to -90 degrees
- turned R5 to -90 degrees
Connections:
- net +5V renamed /V_SYS
- net Net-(J4-PadR) renamed /R
- net Net-(J4-PadT) renamed /T
- net Net-(U6-BAT) renamed /batt
- net Net-(U6-VBUS) renamed /VBUS
- C17 pad 1: +3.3V -> Net-(U3-VDDA)
- R4 pad 1: +3.3V -> /I2C_SCL
- R4 pad 2: /I2C_SCL -> +3.3V
- R5 pad 1: +3.3V -> /I2C_SDA
- R5 pad 2: /I2C_SDA -> +3.3V
- U3 pad 122: unconnected-(U3-PD6-Pad122) -> /CHG_PG
- U3 pad 123: unconnected-(U3-PD7-Pad123) -> /V1P8_EN
- U3 pad 33: +3.3V -> Net-(U3-VDDA)
- U3 pad 8: unconnected-(U3-PC14-Pad8) -> /PD
- U5 pad D4: unconnected-(U5-PD-PadD4) -> /PD
- U5 pad F2: +1V8 -> Net-(L4-Pad1)
- U6 pad 3: GND -> /CHG_PG
- U7 pad 41: unconnected-(U7-GND-Pad41) -> GND
- U7 pad 42: unconnected-(U7-GND-Pad42) -> GND
- U7 pad 43: unconnected-(U7-GND-Pad43) -> GND
- U7 pad 44: unconnected-(U7-GND-Pad44) -> GND
- U9 pad 26: unconnected-(U9-GND-Pad26) -> GND
- U9 pad 28: unconnected-(U9-GND-Pad28) -> GND
- U9 pad 31: unconnected-(U9-GND-Pad31) -> GND
- U9 pad 32: unconnected-(U9-GND-Pad32) -> GND
- U9 pad 33: unconnected-(U9-GND-Pad33) -> GND
Routing:
- net /V1P8_EN: track 12.4 -> 38.8 mm, vias 3 -> 6
- net /CHG_PG: track 0.00 -> 14.6 mm, vias 0 -> 3
- net GND: track 107.8 -> 120.2 mm, vias 90 -> 98
- net Net-(L4-Pad1): track 0.00 -> 9.45 mm, vias 0 -> 2
- net /PD: track 0.00 -> 7.14 mm
- net Net-(U3-VDDA): track 0.00 -> 3.45 mm, vias 0 -> 1
- net +1V8: track 48.4 -> 50.3 mm, vias 6 -> 5
- net +3.3V: track 54.8 -> 56.1 mm, vias 36 -> 35
- net /batt: track 18.3 -> 19.4 mm
- net /temp: track 28.5 -> 27.4 mm
- net Net-(U3-NRST): track 0.50 -> 1.36 mm
- net /CHG_INT: track 34.4 -> 35.2 mm
- net /BLT_RESET: track 15.7 -> 15.1 mm
- net /HPOUTL: track 10.4 -> 9.87 mm
- net Net-(U6-ILIM): track 5.84 -> 5.33 mm
