File: Serene Mini Hardware/Serene Mini.kicad_sch (KiCad schematic)
At the start: 80 parts, among them J1 Conn_Coaxial, J2 Conn_01x06_Socket, J4 AudioJack3_Switch, J5 USB_C_Receptacle_USB2.0_14P, J6 Conn_Coaxial, T1 Transformer_1P_1S, U1 AP7361C-33E, U2 AP2112K-1.8, U3 STM32H753ZITx, U4 ADXL382-1BCCZ-RL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

Commit message: Minor Changes
Parts:
- removed R12: 100kΩ, Resistor_SMD:R_0402_1005Metric, symbol Device:R_Small
- added L3, L4: 600Ω, Inductor_SMD:L_0402_1005Metric, symbol Device:L_Ferrite
- C17: value 0.1uF -> 4.7µF
- U9: value ~ -> SR1120
Connections:
- net +1V8: now also L4.2; no longer U5.F2 (AVDD)
- net +3.3V: now also R4.2, R5.2, L3.2; no longer C17.1, R4.1, R5.1, U3.33 (VDDA)
- net GND: now also U7.41 (GND), U7.42 (GND), U7.43 (GND), U7.44 (GND), U9.26 (GND), U9.28 (GND), U9.31 (GND), U9.32 (GND), U9.33 (GND); no longer U6.3 (PG)
- net I2C_SCL: now also R4.1; no longer R4.2
- net I2C_SDA: now also R5.1; no longer R5.2
- net V1P8_EN: now also U3.123 (PD7)
- net VBUS: now reaches C40.2, J5.A4 (VBUS), J5.A9 (VBUS), J5.B4 (VBUS), J5.B9 (VBUS), U6.18 (VBUS)
- net T: now reaches J4.T, U8.1 (I/O1)
- net R: now reaches J4.R, U8.3 (I/O2)
- net batt: now reaches C1.2, R9.2, TP5.1, U6.8 (BAT)
- net CHG_PG: now reaches U3.122 (PD6)
- net CHG_PG: now also U6.3 (PG)
- net PD: now reaches U3.8 (PC14)
- net PD: now also U5.D4 (PD)
- net +5V renamed V_SYS
- new net: C17.1, L3.1, U3.33 (VDDA)
- new net: L4.1, U5.F2 (AVDD)
Other:
- note added: "Battery and button. Includes button and battery connectors."
- note added: "DSP and VIbration Sensor."
- note added: "Mics and Headphone Jack."
- note added: "Must be a 500mAh battery or larger, if battery is smaller(100mAh to 499mAh) use a 10kΩ resistor must be used."
- note added: "Power. Includes Power Regulator, USB-C port, and Power IC."
- note added: "STM32H7 microcontroller and testpoints to flash firmware."
- note added: "Singal chips, specifically the Bluetooth and UWB Chips."
- note removed: "Must be a 500mAh battery or larger, if smaller battery is used a 10kΩ resistor must be used for a battery of capacity 100mAh to 499mAh"
- moved on the sheet: C1, C10, C11, C12, C13, C14, C15, C16, C17, C18, C19, C2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
